File: Timer_eagle/timer.sch (EAGLE design)
At the start: 21 parts, among them IC1 NE555, IC2 4081N, IC3 4518N, IC4 4070N, K1 G5L, Q1 BC548, Q2 TIP120, X1 SSW-103-02-S-S

Commit message: Projeto final da placa
Parts:
- removed X1: SSW-103-02-S-S, con-samtec:SSW-103-02-S-S
- added JP1, JP2, JP3: (no value), pinhead:PINHD-1X1
Connections:
- net N$19: now also JP1.1; no longer X1-1.1
- net N$20: now also JP2.1; no longer X1-2.1
- net N$21: now also JP3.1; no longer X1-3.1
Changed lines of the file:
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@@
 <part name="P+5" library="supply1" deviceset="VCC" device=""/>
 <part name="GND4" library="supply1" deviceset="GND" device=""/>
-<part name="X1" library="con-samtec" deviceset="SSW-103-02-S-S" device=""/>
 <part name="R5" library="eagle-ltspice" deviceset="R" device="0207/10"/>
 <part name="R6" library="eagle-ltspice" deviceset="R" device="0207/10"/>
@@
 <part name="VSS1" library="supply1" deviceset="VSS" device=""/>
 <part name="SUPPLY1" library="supply2" deviceset="VSS" device=""/>
+<part name="JP1" library="pinhead" deviceset="PINHD-1X1" device=""/>
+<part name="JP2" library="pinhead" deviceset="PINHD-1X1" device=""/>
+<part name="JP3" library="pinhead" deviceset="PINHD-1X1" device=""/>
 </parts>
 <sheets>
@@
 <instance part="P+5" gate="VCC" x="83.82" y="91.44"/>
 <instance part="GND4" gate="1" x="83.82" y="53.34"/>
-<instance part="X1" gate="-1" x="116.84" y="50.8"/>
-<instance part="X1" gate="-2" x="116.84" y="48.26"/>
-<instance part="X1" gate="-3" x="116.84" y="45.72"/>
 <instance part="R5" gate="G$1" x="134.62" y="83.82"/>
 <instance part="R6" gate="G$1" x="152.4" y="71.12" rot="R270"/>
@@
 <instance part="VSS1" gate="G$1" x="30.48" y="91.44"/>
 <instance part="SUPPLY1" gate="G$1" x="35.56" y="93.98"/>
+<instance part="JP1" gate="G$1" x="99.06" y="55.88" rot="MR0"/>
+<instance part="JP2" gate="G$1" x="99.06" y="48.26" rot="MR0"/>
+<instance part="JP3" gate="G$1" x="99.06" y="40.64" rot="MR0"/>
 </instances>
 <busses>
@@
 </segment>
 </net>
-<net name="N$20" class="0">
-<segment>
-<wire x1="137.16" y1="50.8" x2="137.16" y2="55.88" width="0.1524" layer="91"/>
-<wire x1="137.16" y1="55.88" x2="144.78" y2="55.88" width="0.1524" layer="91"/>
-<wire x1="144.78" y1="55.88" x2="144.78" y2="53.34" width="0.1524" layer="91"/>
-<pinref part="K1" gate="2" pin="S"/>
-<wire x1="144.78" y1="53.34" x2="144.78" y2="50.8" width="0.1524" layer="91"/>
-<junction x="144.78" y="53.34"/>
-<wire x1="137.16" y1="50.8" x2="129.54" y2="50.8" width="0.1524" layer="91"/>
-<wire x1="129.54" y1="50.8" x2="129.54" y2="48.26" width="0.1524" layer="91"/>
-<pinref part="X1" gate="-2" pin="1"/>
-<wire x1="129.54" y1="48.26" x2="119.38" y2="48.26" width="0.1524" layer="91"/>
-</segment>
-</net>
 <net name="N$21" class="0">
 <segment>
-<pinref part="X1" gate="-3" pin="1"/>
-<wire x1="119.38" y1="45.72" x2="137.16" y2="45.72" width="0.1524" layer="91"/>
+<wire x1="111.76" y1="45.72" x2="137.16" y2="45.72" width="0.1524" layer="91"/>
 <wire x1="137.16" y1="45.72" x2="137.16" y2="38.1" width="0.1524" layer="91"/>
 <wire x1="137.16" y1="38.1" x2="144.78" y2="38.1" width="0.1524" layer="91"/>
 <pinref part="K1" gate="2" pin="O"/>
 <wire x1="144.78" y1="38.1" x2="144.78" y2="43.18" width="0.1524" layer="91"/>
+<wire x1="111.76" y1="45.72" x2="111.76" y2="40.64" width="0.1524" layer="91"/>
+<pinref part="JP3" gate="G$1" pin="1"/>
+<wire x1="111.76" y1="40.64" x2="101.6" y2="40.64" width="0.1524" layer="91"/>
 </segment>
 </net>
@@
 <wire x1="139.7" y1="83.82" x2="147.32" y2="83.82" width="0.1524" layer="91"/>
 <junction x="139.7" y="83.82"/>
-</segment>
-</net>
-<net name="N$19" class="0">
-<segment>
-<pinref part="K1" gate="2" pin="P"/>
-<wire x1="137.16" y1="48.26" x2="132.08" y2="48.26" width="0.1524" layer="91"/>
-<wire x1="132.08" y1="48.26" x2="132.08" y2="53.34" width="0.1524" layer="91"/>
-<wire x1="132.08" y1="53.34" x2="119.38" y2="53.34" width="0.1524" layer="91"/>
-<pinref part="X1" gate="-1" pin="1"/>
-<wire x1="119.38" y1="53.34" x2="119.38" y2="50.8" width="0.1524" layer="91"/>
 </segment>
 </net>
@@
 </segment>
 </net>
+<net name="N$19" class="0">
+<segment>
+<pinref part="K1" gate="2" pin="P"/>
+<wire x1="137.16" y1="48.26" x2="132.08" y2="48.26" width="0.1524" layer="91"/>
+<wire x1="132.08" y1="48.26" x2="132.08" y2="55.88" width="0.1524" layer="91"/>
+<wire x1="132.08" y1="55.88" x2="101.6" y2="55.88" width="0.1524" layer="91"/>
+<pinref part="JP1" gate="G$1" pin="1"/>
+</segment>
+</net>
+<net name="N$20" class="0">
+<segment>
+<pinref part="K1" gate="2" pin="S"/>
+<wire x1="144.78" y1="53.34" x2="109.22" y2="53.34" width="0.1524" layer="91"/>
+<wire x1="109.22" y1="53.34" x2="109.22" y2="48.26" width="0.1524" layer="91"/>
+<pinref part="JP2" gate="G$1" pin="1"/>
+<wire x1="109.22" y1="48.26" x2="101.6" y2="48.26" width="0.1524" layer="91"/>
+</segment>
+</net>
